File: AVcarrierBoard/AVcarrierBoard.kicad_sch (KiCad schematic)
At the start: 12 parts, among them J1 QuarkRecov, J2 RavenStaging, J3 RavenRecov, J4 Mech_Switch, J5 Mech_Switch, U1 EggfinderMini/FeatherGPS, U2 EggtimerQuark, U3 Blue_Raven, U4 WiFi Switch, U5 WiFi Switch

Commit message: Created PCB, linked 3D step files to footprints, and laid out board (10 inch length)
Parts:
- J1: value QuarkRecov -> MainRecov; footprint COTS_Boards:ScrewTerminals_2828362 -> COTS_Boards:TE_282837-4
- J2: footprint COTS_Boards:ScrewTerminals_2828362 -> COTS_Boards:TE_282837-4
- J3: value RavenRecov -> DrogRecov; footprint COTS_Boards:ScrewTerminals_2828362 -> COTS_Boards:TE_282837-4
- U1: footprint COTS_Boards:EggfinderMini -> COTS_Boards:Featherweight_GPS
- U3: footprint Library:Blue Raven -> COTS_Boards:Blue Raven
- U4, U5: footprint (none) -> COTS_Boards:Eggtime_WiFi_switch
Connections:
- net DROG1: now also J3.1 (Pin_1); no longer J1.3 (Pin_3)
- net DROG2: now also J3.2 (Pin_2); no longer J1.4 (Pin_4)
- net RavenMAIN: now also J1.3 (Pin_3); no longer J3.1 (Pin_1)
- net BATT_1S renamed WIFI_PWR_1S
- net WIFI_PWR_1S: now also J1.4 (Pin_4); no longer J3.2 (Pin_2)
- net BATT_2S renamed WIFI_PWR_2S
Changed lines of the file:
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@@
     )
   )
-  (global_label "BATT_2S" (shape input) (at 104.14 66.04 0) (fields_autoplaced)
-    (effects (font (size 1.27 1.27)) (justify left))
-    (property "Intersheetrefs" "${INTERSHEET_REFS}" (at 114.8056 66.04 0)
-      (effects (font (size 1.27 1.27)) (justify left) hide)
-    )
-  )
-  (global_label "DROG1" (shape input) (at 166.37 74.93 180) (fields_autoplaced)
-    (effects (font (size 1.27 1.27)) (justify right))
-    (property "Intersheetrefs" "${INTERSHEET_REFS}" (at 157.0348 74.93 0)
+  (global_label "WIFI_PWR_2S" (shape input) (at 104.14 66.04 0) (fields_autoplaced)
+    (effects (font (size 1.27 1.27)) (justify left))
+    (property "Intersheetrefs" "${INTERSHEET_REFS}" (at 119.2204 66.04 0)
+      (effects (font (size 1.27 1.27)) (justify left) hide)
+    )
+  )
+  (global_label "RavenMAIN" (shape input) (at 166.37 74.93 180) (fields_autoplaced)
+    (effects (font (size 1.27 1.27)) (justify right))
+    (property "Intersheetrefs" "${INTERSHEET_REFS}" (at 153.2853 74.93 0)
       (effects (font (size 1.27 1.27)) (justify right) hide)
     )
@@
     )
   )
-  (global_label "BATT_1S" (shape input) (at 166.37 113.03 180) (fields_autoplaced)
-    (effects (font (size 1.27 1.27)) (justify right))
-    (property "Intersheetrefs" "${INTERSHEET_REFS}" (at 155.7044 113.03 0)
+  (global_label "WIFI_PWR_1S" (shape input) (at 166.37 113.03 180) (fields_autoplaced)
+    (effects (font (size 1.27 1.27)) (justify right))
+    (property "Intersheetrefs" "${INTERSHEET_REFS}" (at 151.2896 113.03 0)
       (effects (font (size 1.27 1.27)) (justify right) hide)
     )
@@
     )
   )
-  (global_label "RavenMAIN" (shape input) (at 166.37 105.41 180) (fields_autoplaced)
-    (effects (font (size 1.27 1.27)) (justify right))
-    (property "Intersheetrefs" "${INTERSHEET_REFS}" (at 153.2853 105.41 0)
-      (effects (font (size 1.27 1.27)) (justify right) hide)
-    )
-  )
-  (global_label "BATT_1S" (shape input) (at 166.37 90.17 180) (fields_autoplaced)
-    (effects (font (size 1.27 1.27)) (justify right))
-    (property "Intersheetrefs" "${INTERSHEET_REFS}" (at 155.7044 90.17 0)
-      (effects (font (size 1.27 1.27)) (justify right) hide)
-    )
-  )
-  (global_label "DROG2" (shape input) (at 166.37 77.47 180) (fields_autoplaced)
-    (effects (font (size 1.27 1.27)) (justify right))
-    (property "Intersheetrefs" "${INTERSHEET_REFS}" (at 157.0348 77.47 0)
+  (global_label "DROG1" (shape input) (at 166.37 105.41 180) (fields_autoplaced)
+    (effects (font (size 1.27 1.27)) (justify right))
+    (property "Intersheetrefs" "${INTERSHEET_REFS}" (at 157.0348 105.41 0)
+      (effects (font (size 1.27 1.27)) (justify right) hide)
+    )
+  )
+  (global_label "WIFI_PWR_1S" (shape input) (at 166.37 90.17 180) (fields_autoplaced)
+    (effects (font (size 1.27 1.27)) (justify right))
+    (property "Intersheetrefs" "${INTERSHEET_REFS}" (at 151.2896 90.17 0)
+      (effects (font (size 1.27 1.27)) (justify right) hide)
+    )
+  )
+  (global_label "WIFI_PWR_1S" (shape input) (at 166.37 77.47 180) (fields_autoplaced)
+    (effects (font (size 1.27 1.27)) (justify right))
+    (property "Intersheetrefs" "${INTERSHEET_REFS}" (at 151.2896 77.47 0)
       (effects (font (size 1.27 1.27)) (justify right) hide)
     )
@@
     )
   )
-  (global_label "BATT_1S" (shape input) (at 166.37 95.25 180) (fields_autoplaced)
-    (effects (font (size 1.27 1.27)) (justify right))
-    (property "Intersheetrefs" "${INTERSHEET_REFS}" (at 155.7044 95.25 0)
+  (global_label "WIFI_PWR_1S" (shape input) (at 166.37 95.25 180) (fields_autoplaced)
+    (effects (font (size 1.27 1.27)) (justify right))
+    (property "Intersheetrefs" "${INTERSHEET_REFS}" (at 151.2896 95.25 0)
       (effects (font (size 1.27 1.27)) (justify right) hide)
     )
@@
     )
   )
-  (global_label "BATT_1S" (shape input) (at 166.37 107.95 180) (fields_autoplaced)
-    (effects (font (size 1.27 1.27)) (justify right))
-    (property "Intersheetrefs" "${INTERSHEET_REFS}" (at 155.7044 107.95 0)
+  (global_label "DROG2" (shape input) (at 166.37 107.95 180) (fields_autoplaced)
+    (effects (font (size 1.27 1.27)) (justify right))
+    (property "Intersheetrefs" "${INTERSHEET_REFS}" (at 157.0348 107.95 0)
       (effects (font (size 1.27 1.27)) (justify right) hide)
     )
@@
     )
   )
-  (global_label "BATT_2S" (shape input) (at 116.84 85.09 180) (fields_autoplaced)
-    (effects (font (size 1.27 1.27)) (justify right))
-    (property "Intersheetrefs" "${INTERSHEET_REFS}" (at 106.1744 85.09 0)
+  (global_label "WIFI_PWR_2S" (shape input) (at 116.84 85.09 180) (fields_autoplaced)
+    (effects (font (size 1.27 1.27)) (justify right))
+    (property "Intersheetrefs" "${INTERSHEET_REFS}" (at 101.7596 85.09 0)
       (effects (font (size 1.27 1.27)) (justify right) hide)
     )
@@
     )
   )
-  (global_label "BATT_2S" (shape input) (at 116.84 74.93 180) (fields_autoplaced)
-    (effects (font (size 1.27 1.27)) (justify right))
-    (property "Intersheetrefs" "${INTERSHEET_REFS}" (at 106.1744 74.93 0)
+  (global_label "WIFI_PWR_2S" (shape input) (at 116.84 74.93 180) (fields_autoplaced)
+    (effects (font (size 1.27 1.27)) (justify right))
+    (property "Intersheetrefs" "${INTERSHEET_REFS}" (at 101.7596 74.93 0)
       (effects (font (size 1.27 1.27)) (justify right) hide)
     )
@@
     )
   )
-  (global_label "BATT_1S" (shape input) (at 101.6 109.22 0) (fields_autoplaced)
-    (effects (font (size 1.27 1.27)) (justify left))
-    (property "Intersheetrefs" "${INTERSHEET_REFS}" (at 112.2656 109.22 0)
+  (global_label "WIFI_PWR_1S" (shape input) (at 101.6 109.22 0) (fields_autoplaced)
+    (effects (font (size 1.27 1.27)) (justify left))
+    (property "Intersheetrefs" "${INTERSHEET_REFS}" (at 116.6804 109.22 0)
       (effects (font (size 1.27 1.27)) (justify left) hide)
     )
@@
     )
   )
-  (global_label "BATT_1S" (shape input) (at 135.89 116.84 0) (fields_autoplaced)
-    (effects (font (size 1.27 1.27)) (justify left))
-    (property "Intersheetrefs" "${INTERSHEET_REFS}" (at 146.5556 116.84 0)
+  (global_label "WIFI_PWR_1S" (shape input) (at 135.89 116.84 0) (fields_autoplaced)
+    (effects (font (size 1.27 1.27)) (justify left))
+    (property "Intersheetrefs" "${INTERSHEET_REFS}" (at 150.9704 116.84 0)
       (effects (font (size 1.27 1.27)) (justify left) hide)
     )
@@
       (effects (font (size 1.27 1.27)))
     )
-    (property "Footprint" "Library:Blue Raven" (at 123.19 121.92 0)
+    (property "Footprint" "COTS_Boards:Blue Raven" (at 123.19 121.92 0)
       (effects (font (size 1.27 1.27)) hide)
     )
@@
       (effects (font (size 1.27 1.27)) (justify left))
     )
-    (property "Value" "RavenRecov" (at 173.99 110.49 0)
-      (effects (font (size 1.27 1.27)) (justify left))
-    )
-    (property "Footprint" "COTS_Boards:ScrewTerminals_2828362" (at 171.45 107.95 0)
+    (property "Value" "DrogRecov" (at 173.99 110.49 0)
+      (effects (font (size 1.27 1.27)) (justify left))
+    )
+    (property "Footprint" "COTS_Boards:TE_282837-4" (at 171.45 107.95 0)
       (effects (font (size 1.27 1.27)) hide)
     )
@@
       (effects (font (size 1.27 1.27)))
     )
-    (property "Footprint" "" (at 95.25 66.04 0)
+    (property "Footprint" "COTS_Boards:Eggtime_WiFi_switch" (at 95.25 66.04 0)
       (effects (font (size 1.27 1.27)) hide)
     )
@@
       (effects (font (size 1.27 1.27)) (justify left))
     )
-    (property "Value" "QuarkRecov" (at 173.99 74.93 0)
-      (effects (font (size 1.27 1.27)) (justify left))
-    )
-    (property "Footprint" "COTS_Boards:ScrewTerminals_2828362" (at 171.45 72.39 0)
+    (property "Value" "MainRecov" (at 173.99 74.93 0)
+      (effects (font (size 1.27 1.27)) (justify left))
+    )
+    (property "Footprint" "COTS_Boards:TE_282837-4" (at 171.45 72.39 0)
       (effects (font (size 1.27 1.27)) hide)
     )
@@
       (effects (font (size 1.27 1.27)) (justify left))
     )
-    (property "Footprint" "COTS_Boards:ScrewTerminals_2828362" (at 171.45 90.17 0)
+    (property "Footprint" "COTS_Boards:TE_282837-4" (at 171.45 90.17 0)
       (effects (font (size 1.27 1.27)) hide)
     )
@@
       (effects (font (size 1.27 1.27)) (justify right))
     )
-    (property "Footprint" "COTS_Boards:EggfinderMini" (at 123.19 91.44 0)
+    (property "Footprint" "COTS_Boards:Featherweight_GPS" (at 123.19 91.44 0)
       (effects (font (size 1.27 1.27)) hide)
     )
@@
       (effects (font (size 1.27 1.27)))
     )
-    (property "Footprint" "" (at 92.71 109.22 0)
-      (effects (font (size 1.27 1.27)) hide)
-    )
+    (property "Footprint" "COTS_Boards:Eggtime_WiFi_switch" (at 92.71 109.22 0)
+      (effects (font (size 1.27 1.27)) hide)
+    )

Commit message: ok ok
Parts:
- removed J2: RavenStaging, COTS_Boards:TE_282837-4, symbol Connector:Screw_Terminal_01x04
- added J6: 462070006, CON_462070006, symbol COTS_boards:462070006
Connections:
- net GND: no longer BT2.2 (-), U3.2 (Gnd), U4.2 (Batt-), U4.4 (Out-)
- net Raven3RD: now also J6.3, J6.5
- net Raven4TH: now also J6.1
- net WIFI_PWR_1S: now also J6.2, J6.4, J6.6
- new net GND2: BT2.2 (-), U3.2 (Gnd), U4.2 (Batt-), U4.4 (Out-)
Changed lines of the file:
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@@
 (kicad_sch (version 20230121) (generator eeschema)
   (paper "A4")
-  (wire (pts (xy 142.24 114.3) (xy 142.24 120.65))
-    (stroke (width 0) (type default))
-  )
-  (wire (pts (xy 135.89 114.3) (xy 142.24 114.3))
-    (stroke (width 0) (type default))
-  )
   (global_label "+3V8" (shape input) (at 50.8 114.3 180) (fields_autoplaced)
     (effects (font (size 1.27 1.27)) (justify right))
@@
     )
   )
+  (global_label "Raven3RD" (shape input) (at 166.37 97.79 180) (fields_autoplaced)
+    (effects (font (size 1.27 1.27)) (justify right))
+    (property "Intersheetrefs" "${INTERSHEET_REFS}" (at 154.0111 97.79 0)
+      (effects (font (size 1.27 1.27)) (justify right) hide)
+    )
+  )
   (global_label "RavenMAIN" (shape input) (at 166.37 74.93 180) (fields_autoplaced)
     (effects (font (size 1.27 1.27)) (justify right))
@@
     )
   )
+  (global_label "GND2" (shape input) (at 83.82 111.76 180) (fields_autoplaced)
+    (effects (font (size 1.27 1.27)) (justify right))
+    (property "Intersheetrefs" "${INTERSHEET_REFS}" (at 75.7548 111.76 0)
+      (effects (font (size 1.27 1.27)) (justify right) hide)
+    )
+  )
   (global_label "RavenAPO" (shape input) (at 166.37 110.49 180) (fields_autoplaced)
     (effects (font (size 1.27 1.27)) (justify right))
@@
     )
   )
+  (global_label "GND2" (shape input) (at 135.89 114.3 0) (fields_autoplaced)
+    (effects (font (size 1.27 1.27)) (justify left))
+    (property "Intersheetrefs" "${INTERSHEET_REFS}" (at 143.9552 114.3 0)
+      (effects (font (size 1.27 1.27)) (justify left) hide)
+    )
+  )
   (global_label "Raven3RD" (shape input) (at 166.37 92.71 180) (fields_autoplaced)
     (effects (font (size 1.27 1.27)) (justify right))
@@
     )
   )
+  (global_label "WIFI_PWR_1S" (shape input) (at 166.37 100.33 180) (fields_autoplaced)
+    (effects (font (size 1.27 1.27)) (justify right))
+    (property "Intersheetrefs" "${INTERSHEET_REFS}" (at 151.2896 100.33 0)
+      (effects (font (size 1.27 1.27)) (justify right) hide)
+    )
+  )
   (global_label "DROG1" (shape input) (at 132.08 71.12 0) (fields_autoplaced)
     (effects (font (size 1.27 1.27)) (justify left))
@@
     )
   )
+  (global_label "GND2" (shape input) (at 86.36 130.81 270) (fields_autoplaced)
+    (effects (font (size 1.27 1.27)) (justify right))
+    (property "Intersheetrefs" "${INTERSHEET_REFS}" (at 86.36 138.8752 90)
+      (effects (font (size 1.27 1.27)) (justify right) hide)
+    )
+  )
   (global_label "MAIN1" (shape input) (at 132.08 66.04 0) (fields_autoplaced)
     (effects (font (size 1.27 1.27)) (justify left))
@@
     (effects (font (size 1.27 1.27)) (justify left))
     (property "Intersheetrefs" "${INTERSHEET_REFS}" (at 150.9704 116.84 0)
+      (effects (font (size 1.27 1.27)) (justify left) hide)
+    )
+  )
+  (global_label "GND2" (shape input) (at 101.6 111.76 0) (fields_autoplaced)
+    (effects (font (size 1.27 1.27)) (justify left))
+    (property "Intersheetrefs" "${INTERSHEET_REFS}" (at 109.6652 111.76 0)
       (effects (font (size 1.27 1.27)) (justify left) hide)
     )
@@
     )
   )
-  (symbol (lib_id "power:GND") (at 83.82 111.76 0) (unit 1)
-    (in_bom yes) (on_board yes) (dnp no) (fields_autoplaced)
-    (property "Reference" "#PWR08" (at 83.82 118.11 0)
-      (effects (font (size 1.27 1.27)) hide)
-    )
-    (property "Value" "GND" (at 83.82 116.84 0)
-      (effects (font (size 1.27 1.27)))
-    )
-    (property "Footprint" "" (at 83.82 111.76 0)
-      (effects (font (size 1.27 1.27)) hide)
-    )
-    (property "Datasheet" "" (at 83.82 111.76 0)
-      (effects (font (size 1.27 1.27)) hide)
-    )
-    (pin "1")
-    (instances
-      (project "AVcarrierBoard"
-        (path "/7d4c9aa4-eccf-4732-8f5d-af2c3b6d9138"
-          (reference "#PWR08") (unit 1)
-        )
-      )
-    )
-  )
   (symbol (lib_id "power:GND") (at 116.84 87.63 0) (unit 1)
     (in_bom yes) (on_board yes) (dnp no) (fields_autoplaced)
@@
     )
   )
-  (symbol (lib_id "power:GND") (at 101.6 111.76 0) (unit 1)
-    (in_bom yes) (on_board yes) (dnp no) (fields_autoplaced)
-    (property "Reference" "#PWR09" (at 101.6 118.11 0)
-      (effects (font (size 1.27 1.27)) hide)
-    )
-    (property "Value" "GND" (at 101.6 116.84 0)
-      (effects (font (size 1.27 1.27)))
-    )
-    (property "Footprint" "" (at 101.6 111.76 0)
-      (effects (font (size 1.27 1.27)) hide)
-    )
-    (property "Datasheet" "" (at 101.6 111.76 0)
-      (effects (font (size 1.27 1.27)) hide)
-    )
-    (pin "1")
-    (instances
-      (project "AVcarrierBoard"
-        (path "/7d4c9aa4-eccf-4732-8f5d-af2c3b6d9138"
-          (reference "#PWR09") (unit 1)
-        )
-      )
-    )
-  )
   (symbol (lib_id "Connector:Screw_Terminal_01x04") (at 171.45 72.39 0) (unit 1)
     (in_bom yes) (on_board yes) (dnp no) (fields_autoplaced)
@@
         (path "/7d4c9aa4-eccf-4732-8f5d-af2c3b6d9138"
           (reference "#PWR01") (unit 1)
-        )
-      )
-    )
-  )
-  (symbol (lib_id "power:GND") (at 86.36 130.81 0) (unit 1)
-    (in_bom yes) (on_board yes) (dnp no) (fields_autoplaced)
-    (property "Reference" "#PWR02" (at 86.36 137.16 0)
-      (effects (font (size 1.27 1.27)) hide)
-    )
-    (property "Value" "GND" (at 86.36 135.89 0)
-      (effects (font (size 1.27 1.27)))
-    )
-    (property "Footprint" "" (at 86.36 130.81 0)
-      (effects (font (size 1.27 1.27)) hide)
-    )
-    (property "Datasheet" "" (at 86.36 130.81 0)
-      (effects (font (size 1.27 1.27)) hide)
-    )
-    (pin "1")
-    (instances
-      (project "AVcarrierBoard"
-        (path "/7d4c9aa4-eccf-4732-8f5d-af2c3b6d9138"
-          (reference "#PWR02") (unit 1)
-        )
-      )
-    )
-  )
-  (symbol (lib_id "Connector:Screw_Terminal_01x04") (at 171.45 90.17 0) (unit 1)
-    (in_bom yes) (on_board yes) (dnp no) (fields_autoplaced)
-    (property "Reference" "J2" (at 173.99 90.17 0)
-      (effects (font (size 1.27 1.27)) (justify left))
-    )
-    (property "Value" "RavenStaging" (at 173.99 92.71 0)
-      (effects (font (size 1.27 1.27)) (justify left))
-    )
-    (property "Footprint" "COTS_Boards:TE_282837-4" (at 171.45 90.17 0)
-      (effects (font (size 1.27 1.27)) hide)
-    )
-    (property "Datasheet" "~" (at 171.45 90.17 0)
-      (effects (font (size 1.27 1.27)) hide)
-    )
-    (pin "4")
-    (pin "3")
-    (pin "2")
-    (pin "1")
-    (instances
-      (project "AVcarrierBoard"
-        (path "/7d4c9aa4-eccf-4732-8f5d-af2c3b6d9138"
-          (reference "J2") (unit 1)
         )
       )
@@
     )
   )
-  (symbol (lib_id "power:GND") (at 142.24 120.65 0) (unit 1)
-    (in_bom yes) (on_board yes) (dnp no) (fields_autoplaced)
-    (property "Reference" "#PWR07" (at 142.24 127 0)
-      (effects (font (size 1.27 1.27)) hide)
-    )
-    (property "Value" "GND" (at 142.24 125.73 0)
-      (effects (font (size 1.27 1.27)))
-    )
-    (property "Footprint" "" (at 142.24 120.65 0)
-      (effects (font (size 1.27 1.27)) hide)
-    )
-    (property "Datasheet" "" (at 142.24 120.65 0)
-      (effects (font (size 1.27 1.27)) hide)
-    )
-    (pin "1")
-    (instances
-      (project "AVcarrierBoard"
-        (path "/7d4c9aa4-eccf-4732-8f5d-af2c3b6d9138"
-          (reference "#PWR07") (unit 1)
-        )
-      )
+  (symbol (lib_id "COTS_boards:462070006") (at 166.37 87.63 0) (unit 1)
+    (in_bom yes) (on_board yes) (dnp no) (fields_autoplaced)
+    (property "Reference" "J6" (at 180.34 92.71 0)
+      (effects (font (size 1.524 1.524)) (justify left))
+    )
+    (property "Value" "462070006" (at 180.34 95.25 0)
+      (effects (font (size 1.524 1.524)) (justify left))
+    )
+    (property "Footprint" "CON_462070006" (at 166.37 87.63 0)
+      (effects (font (size 1.27 1.27) italic) hide)
+    )
+    (property "Datasheet" "462070006" (at 166.37 87.63 0)
+      (effects (font (size 1.27 1.27) italic) hide)
+    )
+    (pin "1")
+    (pin "4")
+    (pin "5")
+    (pin "2")
+    (pin "6")
+    (pin "3")
+    (instances
+      (project "AVcarrierBoard"
+        (path "/7d4c9aa4-eccf-4732-8f5d-af2c3b6d9138"
+          (reference "J6") (unit 1)
+        )
+      )
