File: AVcarrierBoard/AVcarrierBoard.kicad_pcb (KiCad board)
At the start: 4 copper layers, 253.6 x 59 mm, 16 parts, among them J1 Mech_Switch, J2 Mech_Switch, J3 MainRecov, J4 DrogRecov, J5 Staging, J6 Mech_Switch, U2 WiFi Switch, U3 EggtimerQuantum, U4 EggfinderMini/FeatherGPS, U5 Blue_Raven

Commit message: Added logo and creator names. Need a more creative name plz
Parts:
- added G***: LOGO, LOGO, F.Cu at (260.2, 119.0)
- added G***: LOGO, LOGO, B.Cu at (224.8, 118.8)
Other:
- board text added: "Annabelle Jayadinata, Sam Chen, Ethan Brinser"

Commit message: Updated author names and added missing footprint
Other:
- board text added: "Annabelle Jayadinata, Sam Chen, Ethan Brinser, Victor Huynh"
- board text removed: "Annabelle Jayadinata, Sam Chen, Ethan Brinser"
Changed lines of the file:
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@@
     (effects (font (size 3 3) (thickness 0.15)) (justify left bottom mirror))
   )
-  (gr_text "Annabelle Jayadinata, Sam Chen, Ethan Brinser" (at 265.2776 121.8692) (layer "B.SilkS")
-    (effects (font (size 1 1) (thickness 0.15)) (justify left bottom mirror))
+  (gr_text "Annabelle Jayadinata, Sam Chen, Ethan Brinser, Victor Huynh" (at 265.2776 121.8692) (layer "B.SilkS")
+    (effects (font (size 0.75 0.75) (thickness 0.125)) (justify left bottom mirror))
   )
   (via (at 243.2812 80.772) (size 3) (drill 1) (layers "F.Cu" "B.Cu") (free) (net 1))

Commit message: Rerouted footprint directory
Parts:
- J1, J2: footprint Connector_PinHeader_2.54mm:PinHeader_1x02_P2.97mm_Vertical -> 2.97mmConnector:PinHeader_1x02_P2.97mm_Vertical
- moved G*** 1.02 mm to (223.8, 118.8)
Changed lines of the file:
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@@
       (stroke (width 0) (type solid)) (fill solid) (layer "F.SilkS"))
   )
-  (footprint "Connector_PinHeader_2.54mm:PinHeader_1x02_P2.97mm_Vertical" (layer "F.Cu")
+  (footprint "2.97mmConnector:PinHeader_1x02_P2.97mm_Vertical" (layer "F.Cu")
     (at 144.4702 88.7984 90)
     (descr "Through hole straight pin header, 1x02, 2.54mm pitch, single row")
@@
         (effects (font (size 1 1) (thickness 0.15)))
     )
+    (fp_text user "PTH_DRILL_SIZE:_1.8_MM,_TOL:_+0.05/-0.05" (at -4.199999 8.83 90 unlocked) (layer "Cmts.User")
+        (effects (font (size 1 1) (thickness 0.15)))
+    )
     (fp_text user "NPTH_DRILL_SIZE:_3.0_MM,_TOL:_+0.03/-0.03" (at -4.199999 11.37 90 unlocked) (layer "Cmts.User")
-        (effects (font (size 1 1) (thickness 0.15)))
-    )
-    (fp_text user "PTH_DRILL_SIZE:_1.8_MM,_TOL:_+0.05/-0.05" (at -4.199999 8.83 90 unlocked) (layer "Cmts.User")
         (effects (font (size 1 1) (thickness 0.15)))
     )
@@
       (net 14 "GND2") (pinfunction "Out-") (pintype "power_out"))
   )
-  (footprint "Connector_PinHeader_2.54mm:PinHeader_1x02_P2.97mm_Vertical" (layer "B.Cu")
+  (footprint "2.97mmConnector:PinHeader_1x02_P2.97mm_Vertical" (layer "B.Cu")
     (at 149.4536 101.4426 180)
     (descr "Through hole straight pin header, 1x02, 2.54mm pitch, single row")
@@
   )
   (footprint "LOGO" (layer "B.Cu")
-    (at 224.79 118.8212 180)
+    (at 223.774 118.8212 180)
     (attr board_only exclude_from_pos_files exclude_from_bom)
     (fp_text reference "G***" (at 0 0) (layer "B.SilkS") hide
@@
   )
   (gr_text "Annabelle Jayadinata, Sam Chen, Ethan Brinser, Victor Huynh" (at 265.2776 121.8692) (layer "B.SilkS")
-    (effects (font (size 0.75 0.75) (thickness 0.125)) (justify left bottom mirror))
+    (effects (font (size 0.8 0.8) (thickness 0.125)) (justify left bottom mirror))
   )
   (via (at 243.2812 80.772) (size 3) (drill 1) (layers "F.Cu" "B.Cu") (free) (net 1))

Commit message: Fixed errors and modified board based on comments made by Ethan on Mar 30
Routing:
- net +7.5V: track 39.0 -> 125.6 mm, vias 1 -> 0
- net Raven3RD: track 61.9 -> 76.5 mm
- net GND: track 12.5 -> 22.9 mm, vias 1 -> 2
- net COTSWIFI+: track 43.0 -> 35.7 mm
Other:
- board text added: "EGGDROG"
- board text added: "EGGMAIN"
- board text added: "MOTOR1"
- board text added: "MOTOR2"
- board text added: "RAVDROG"
- board text added: "RAVMAIN"
- board text added: "STAGING1"
- board text added: "STAGING2"

Commit message: final edits made, order placed
Connections:
- BT1 pad 2: GND -> unconnected-(BT1-middle-Pad2)
Routing:
- net +7.5V: track 125.6 -> 39.0 mm
- net unconnected-(BT1-middle-Pad2): track 0.00 -> 19.1 mm
- net GND: track 22.9 -> 12.2 mm, vias 2 -> 1
Changed lines of the file:
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@@
       (plot_on_all_layers_selection 0x0000000_00000000)
       (disableapertmacros false)
-      (usegerberextensions false)
-      (usegerberattributes true)
-      (usegerberadvancedattributes true)
-      (creategerberjobfile true)
+      (usegerberextensions true)
+      (usegerberattributes false)
+      (usegerberadvancedattributes false)
+      (creategerberjobfile false)
       (dashed_line_dash_ratio 12.000000)
       (dashed_line_gap_ratio 3.000000)
@@
       (psa4output false)
       (plotreference true)
-      (plotvalue true)
+      (plotvalue false)
       (plotinvisibletext false)
       (sketchpadsonfab false)
-      (subtractmaskfromsilk false)
+      (subtractmaskfromsilk true)
       (outputformat 1)
       (mirror false)
-      (drillshape 1)
+      (drillshape 0)
       (scaleselection 1)
-      (outputdirectory "")
+      (outputdirectory "Gerbers 0401/")
     )
   )
@@
   (net 15 "RavenMotIgnition")
   (net 16 "PWR_2S")
+  (net 17 "unconnected-(BT1-middle-Pad2)")
   (footprint "LOGO" (layer "F.Cu")
     (at 260.2484 119.0244)
@@
     (property "ki_keywords" "connector")
     (attr through_hole)
-    (fp_text reference "J5" (at -4.199999 -13.97 90 unlocked) (layer "F.SilkS")
+    (fp_text reference "J5" (at -4.199999 -17 90 unlocked) (layer "F.SilkS")
         (effects (font (size 1 1) (thickness 0.15)))
     )
-    (fp_text value "Staging" (at -4.199999 -13.97 90 unlocked) (layer "F.Fab")
+    (fp_text value "Staging" (at -4.199999 -13.97 90 unlocked) (layer "F.Fab") hide
         (effects (font (size 1 1) (thickness 0.15)))
     )
@@
         (effects (font (size 1 1) (thickness 0.15)))
     )
-    (fp_text user "${REFERENCE}" (at -4.199999 -13.97 90 unlocked) (layer "F.Fab")
-        (effects (font (size 1 1) (thickness 0.15)))
-    )
-    (fp_text user "462070006" (at -4.199999 -17.839999 90 unlocked) (layer "F.Fab")
+    (fp_text user "${REFERENCE}" (at -4.199999 -16 90 unlocked) (layer "F.Fab")
         (effects (font (size 1 1) (thickness 0.15)))
     )
@@
     (pad "1" smd rect (at -39.33 -9.555) (size 7.34 6.35) (layers "F.Cu" "F.Paste" "F.Mask")
       (net 8 "+7.5V") (pinfunction "+") (pintype "passive") (solder_mask_margin 0.102))
-    (pad "1" smd rect (at 39.33 9.555) (size 7.34 6.35) (layers "F.Cu" "F.Paste" "F.Mask")
-      (net 8 "+7.5V") (pinfunction "+") (pintype "passive") (solder_mask_margin 0.102))
-    (pad "2" smd rect (at -39.33 9.555) (size 7.34 6.35) (layers "F.Cu" "F.Paste" "F.Mask")
-      (net 2 "GND") (pinfunction "-") (pintype "passive") (solder_mask_margin 0.102))
     (pad "2" smd rect (at 39.33 -9.555) (size 7.34 6.35) (layers "F.Cu" "F.Paste" "F.Mask")
+      (net 17 "unconnected-(BT1-middle-Pad2)") (pinfunction "middle") (pintype "passive+no_connect") (solder_mask_margin 0.102))
+    (pad "3" smd rect (at -39.33 9.555) (size 7.34 6.35) (layers "F.Cu" "F.Paste" "F.Mask")
       (net 2 "GND") (pinfunction "-") (pintype "passive") (solder_mask_margin 0.102))
+    (pad "4" smd rect (at 39.33 9.555) (size 7.34 6.35) (layers "F.Cu" "F.Paste" "F.Mask")
+      (net 17 "unconnected-(BT1-middle-Pad2)") (pinfunction "middle") (pintype "passive+no_connect") (solder_mask_margin 0.102))
     (model "${KIPRJMOD}/1048P--3DModel-STEP-56544.STEP"
       (offset (xyz 0 0 7))
@@
     (effects (font (size 1 1) (thickness 0.15)) (justify left bottom))
   )
-  (gr_text "MOTOR1" (at 34.3408 82.4992) (layer "F.SilkS")
+  (gr_text "MOTOR1" (at 34.4932 82.7024) (layer "F.SilkS")
     (effects (font (size 1 1) (thickness 0.15)) (justify right bottom))
   )
@@
   (segment (start 235.712 80.772) (end 234.315 79.375) (width 2.5) (layer "B.Cu") (net 1))
   (segment (start 243.2812 80.772) (end 235.712 80.772) (width 2.5) (layer "B.Cu") (net 1))
-  (segment (start 255.1638 78.075) (end 252.1204 75.0316) (width 2.5) (layer "F.Cu") (net 2))
-  (segment (start 260.65 78.075) (end 255.1638 78.075) (width 2.5) (layer "F.Cu") (net 2))
-  (segment (start 252.0696 75.0316) (end 251.46 74.422) (width 2.5) (layer "F.Cu") (net 2))
   (segment (start 181.99 97.185) (end 175.865 97.185) (width 2.5) (layer "F.Cu") (net 2))
   (segment (start 175.865 97.185) (end 171.6024 101.4476) (width 2.5) (layer "F.Cu") (net 2))
-  (segment (start 252.1204 75.0316) (end 252.0696 75.0316) (width 2.5) (layer "F.Cu") (net 2))
   (via (at 171.6024 101.4476) (size 3) (drill 1.5) (layers "F.Cu" "B.Cu") (net 2))
-  (via (at 251.46 74.422) (size 3) (drill 1.5) (layers "F.Cu" "B.Cu") (net 2))
   (segment (start 109.965 108.06) (end 117.275 108.06) (width 2.5) (layer "F.Cu") (net 3))
   (segment (start 99.695 97.79) (end 109.965 108.06) (width 2.5) (layer "F.Cu") (net 3))
@@
   (segment (start 149.4536 96.4692) (end 149.4536 101.4426) (width 2.5) (layer "In1.Cu") (net 7))
   (segment (start 168.7068 81.1784) (end 155.0602 81.1784) (width 2.5) (layer "F.Cu") (net 8))
-  (segment (start 224.7854 78.075) (end 243.8954 97.185) (width 2.5) (layer "F.Cu") (net 8))
-  (segment (start 181.99 78.075) (end 224.7854 78.075) (width 2.5) (layer "F.Cu") (net 8))
-  (segment (start 243.8954 97.185) (end 260.65 97.185) (width 2.5) (layer "F.Cu") (net 8))
   (segment (start 181.99 78.075) (end 171.8102 78.075) (width 2.5) (layer "F.Cu") (net 8))
   (segment (start 155.0602 81.1784) (end 147.4402 88.7984) (width 2.5) (layer "F.Cu") (net 8))
@@
   (segment (start 125.7862 94.127) (end 56.2302 94.127) (width 2.5) (layer "B.Cu") (net 15))
   (segment (start 52.7812 90.678) (end 48.105367 90.678) (width 2.5) (layer "B.Cu") (net 15))
+  (segment (start 260.65 78.075) (end 260.65 97.185) (width 2.5) (layer "F.Cu") (net 17))
   (zone (net 16) (net_name "PWR_2S") (layer "F.Cu") (hatch edge 0.5)
     (connect_pads (clearance 0.5))
